Commit message: started prediction node, held items likelihood

File: src/chassis/description/lidar.xacro (robot description, xacro)
@@ -6,5 +6,5 @@
         <parent link="chassis_link"/>
         <child link="lidar_link"/>
-        <origin xyz="0.2 0 0.13442"/>
+        <origin xyz="0.2 0 0.13442" rpy="0 0 3.14159"/>
     </joint>
     <link name="lidar_link">
