Commit message: started on ros2_control

File: src/chassis/description/camera.xacro (robot description, xacro)
@@ -1,4 +1,5 @@
 <?xml version="1.0"?>
 <robot xmlns:xacro="http://www.ros.org/wiki/xacro">
+     <xacro:include filename="inertial_macros.xacro"/>
     <joint name="stick_joint" type="fixed">
         <parent link="chassis_link"/>
@@ -13,4 +14,7 @@
             <material name="black"/>
         </visual>
+        <xacro:inertial_box mass="0.1" x="0.02" y="0.02" z="0.9">
+            <origin xyz="0 0 0" rpy="0 0 0"/>
+        </xacro:inertial_box>
     </link>
     <!-- CAMERA -->
@@ -27,4 +31,35 @@
             <material name="red"/>
         </visual>
+        <xacro:inertial_box mass="0.2" x="0.0076" y="0.1574" z="0.0758">
+            <origin xyz="0 0 0" rpy="0 0 0"/>
+        </xacro:inertial_box>
     </link>
+    <joint name="camera_optical_joint" type="fixed">
+        <parent link="camera_link"/>
+        <child link="camera_optical_link"/>
+        <origin xyz="0 0 0" rpy="-1.5707963267948966 0 -1.5707963267948966"/>
+    </joint>
+    <link name="camera_optical_link"></link>
+    <gazebo reference="camera_link">
+        <material>Gazebo/Red</material>
+        <sensor name="camera" type="camera">
+            <update_rate>10</update_rate>
+            <visualize>true</visualize>
+            <camera>
+                <camera_info_topic>camera/camera_info</camera_info_topic>
+                <horizontal_fov>1.0472</horizontal_fov>
+                <image>
+                    <width>640</width>
+                    <height>480</height>
+                    <format>R8G8B8</format>
+                </image>
+                <clip>
+                    <near>0.05</near>
+                    <far>8.0</far>
+                </clip>
+            </camera>
+            <topic>camera/image_raw</topic>
+            <gz_frame_id>camera_optical_link</gz_frame_id>
+        </sensor>
+    </gazebo>
 </robot>

File: src/chassis/description/chassis.urdf.xacro (robot description, xacro)
@@ -1,5 +1,12 @@
 <?xml version="1.0"?>
 <robot xmlns:xacro="http://www.ros.org/wiki/xacro"  name="robot">
+    <xacro:arg name="use_ros2_control" default="true"/>
     <xacro:include filename="chassis_core.xacro"/>
+    <xacro:if value="$(arg use_ros2_control)">
+        <xacro:include filename="ros2_control.xacro"/>
+    </xacro:if>
+    <xacro:if value="$(arg use_ros2_control)">
+        <xacro:include filename="gazebo_control.xacro"/>
+    </xacro:if>
     <xacro:include filename="lidar.xacro"/>
     <xacro:include filename="camera.xacro"/>

File: src/chassis/description/chassis_core.xacro (robot description, xacro)
@@ -39,4 +39,7 @@
             </geometry>
         </collision>
+        <xacro:inertial_box mass="0.5" x="0.2667" y="0.1651" z="0.127">
+            <origin xyz="0.13335 0 0.0635" rpy="0 0 0"/>
+        </xacro:inertial_box>
     </link>
     <!-- LEFT WHEEL LINK -->
@@ -59,4 +62,7 @@
             </geometry>
         </collision>
+        <xacro:inertial_cylinder mass="0.1" length="0.027" radius="0.035">
+            <origin xyz="0 0 0" rpy="0 0 0"/>
+        </xacro:inertial_cylinder>
     </link>
     <!-- RIGHT WHEEL LINK -->
@@ -79,4 +85,7 @@
             </geometry>
         </collision>
+        <xacro:inertial_cylinder mass="0.1" length="0.027" radius="0.035">
+            <origin xyz="0 0 0" rpy="0 0 0"/>
+        </xacro:inertial_cylinder>
     </link>
     <!-- CASTER WHEEL LINK -->
@@ -99,4 +108,7 @@
             <material name="black"/>
         </collision>
+        <xacro:inertial_sphere mass="0.1" radius="0.035">
+            <origin xyz="0 0 0" rpy="0 0 0"/>
+        </xacro:inertial_sphere>
     </link>
 </robot>

File: src/chassis/description/lidar.xacro (robot description, xacro)
@@ -1,4 +1,5 @@
 <?xml version="1.0"?>
 <robot xmlns:xacro="http://www.ros.org/wiki/xacro">
+    <xacro:include filename="inertial_macros.xacro"/>
     <!-- LIDAR -->
     <joint name="lidar_joint" type="fixed">
@@ -14,4 +15,31 @@
             <material name="red"/>
         </visual>
+        <xacro:inertial_cylinder mass="0.140" length="0.025" radius="0.035">
+            <origin xyz="0 0 0" rpy="0 0 0"/>
+        </xacro:inertial_cylinder>
     </link>
+    <gazebo reference="lidar_link">
+        <material>Gazebo/Red</material>
+        <sensor name="lidar_sensor" type="gpu_lidar">
+            <update_rate>10</update_rate>
+            <visualize>true</visualize>
+            <lidar>
+                <scan>
+                    <horizontal>
+                        <samples>360</samples>
+                        <resolution>1</resolution>
+                        <min_angle>-3.14159</min_angle>
+                        <max_angle>3.14159</max_angle>
+                    </horizontal>
+                </scan>
+                <range>
+                    <min>0.1</min>
+                    <max>10.0</max>
+                    <!-- <resolution>0.01</resolution> -->
+                </range>
+            </lidar>
+            <topic>scan</topic>
+            <gz_frame_id>lidar_link</gz_frame_id>
+        </sensor>
+    </gazebo>
 </robot>

Commit message: flipped xacro model

File: src/chassis/description/camera.xacro (robot description, xacro)
@@ -1,3 +1,3 @@
-<?xml version="1.0"?>
+<!-- <?xml version="1.0"?>
 <robot xmlns:xacro="http://www.ros.org/wiki/xacro">
      <xacro:include filename="inertial_macros.xacro"/>
@@ -63,3 +63,3 @@
         </sensor>
     </gazebo>
-</robot>
+</robot> -->

File: src/chassis/description/chassis.urdf.xacro (robot description, xacro)
@@ -10,4 +10,4 @@
     </xacro:if> -->
     <xacro:include filename="lidar.xacro"/>
-    <xacro:include filename="camera.xacro"/>
+    <!-- <xacro:include filename="camera.xacro"/> -->
 </robot>

File: src/chassis/description/chassis_core.xacro (robot description, xacro)
@@ -29,9 +29,9 @@
         <parent link="base_link"/>
         <child link="chassis_link"/>
-        <origin xyz="-0.0508 0 0" rpy="0 0 0"/> <!-- Offset the chassis slightly back by 5.08cm-->
+        <origin xyz="0.0508 0 0" rpy="0 0 0"/> <!-- Offset the chassis slightly back by 5.08cm-->
     </joint>
     <link name="chassis_link">
         <visual>
-            <origin xyz="0.13462 0 0.06096" rpy="0 0 0"/>
+            <origin xyz="-0.13462 0 0.06096" rpy="0 0 0"/>
             <geometry>
                 <box size="0.26924 0.1524 0.12192"/>
@@ -40,5 +40,5 @@
         </visual>
         <collision>
-            <origin xyz="0.13462 0 0.06096" rpy="0 0 0"/>
+            <origin xyz="-0.13462 0 0.06096" rpy="0 0 0"/>
             <geometry>
                 <box size="0.26924 0.1524 0.12192"/>
@@ -46,5 +46,5 @@
         </collision>
         <xacro:inertial_box mass="0.5" x="0.26924" y="0.1524" z="0.12192">
-            <origin xyz="0.13462 0 0.06096" rpy="0 0 0"/>
+            <origin xyz="-0.13462 0 0.06096" rpy="0 0 0"/>
         </xacro:inertial_box>
     </link>
@@ -53,6 +53,6 @@
         <parent link="base_link"/>
         <child link="left_wheel_link"/>
-        <origin xyz="0 0.09144 -0.0127" rpy="-1.5707963267948966 0 0"/> <!-- Rotate wheel -->
-        <axis xyz="0 0 1"/>
+        <origin xyz="0 -0.09144 -0.0127" rpy="-1.5707963267948966 0 0"/> <!-- Rotate wheel -->
+        <axis xyz="0 0 -1"/>
     </joint>
     <link name="left_wheel_link">
@@ -76,6 +76,6 @@
         <parent link="base_link"/>
         <child link="right_wheel_link"/>
-        <origin xyz="0 -0.09144 -0.0127" rpy="1.5707963267948966 0 0"/> <!-- Rotate wheel -->
-        <axis xyz="0 0 -1"/>
+        <origin xyz="0 0.09144 -0.0127" rpy="1.5707963267948966 0 0"/> <!-- Rotate wheel -->
+        <axis xyz="0 0 1"/>
     </joint>
     <link name="right_wheel_link">
@@ -99,5 +99,5 @@
         <parent link="base_link"/>
         <child link="caster_wheel_link"/>
-        <origin xyz="0.15 0 0" rpy="0 0 0"/>
+        <origin xyz="-0.15 0 0" rpy="0 0 0"/>
     </joint>
     <link name="caster_wheel_link">

File: src/chassis/description/lidar.xacro (robot description, xacro)
@@ -6,5 +6,5 @@
         <parent link="base_link"/>
         <child link="lidar_link"/>
-        <origin xyz="0.15 0 0.13442" rpy="0 0 3.14159"/>
+        <origin xyz="-0.12 0 0.13442" rpy="0 0 0"/>
     </joint>
     <link name="lidar_link">
