Commit message: fixed serial communication

File: src/chassis/description/chassis.urdf.xacro (robot description, xacro)
@@ -1,12 +1,12 @@
 <?xml version="1.0"?>
 <robot xmlns:xacro="http://www.ros.org/wiki/xacro"  name="robot">
-    <xacro:arg name="use_ros2_control" default="true"/>
+    <!-- <xacro:arg name="use_ros2_control" default="true"/> -->
     <xacro:include filename="chassis_core.xacro"/>
-    <xacro:if value="$(arg use_ros2_control)">
+    <!-- <xacro:if value="$(arg use_ros2_control)"> -->
         <xacro:include filename="ros2_control.xacro"/>
-    </xacro:if>
-    <xacro:if value="$(arg use_ros2_control)">
+    <!-- </xacro:if> -->
+    <!-- <xacro:if value="$(arg use_ros2_control)">
         <xacro:include filename="gazebo_control.xacro"/>
-    </xacro:if>
+    </xacro:if> -->
     <xacro:include filename="lidar.xacro"/>
     <xacro:include filename="camera.xacro"/>

File: src/chassis/description/ros2_control.xacro (robot description, xacro)
@@ -4,10 +4,10 @@
         <ros2_control name="RealRobot" type="system">
             <hardware>
-                <plugin>diffdrive_arduino_hardware/DiffDriveArduinoHardware</plugin>
+                <plugin>diffdrive_arduino/DiffDriveArduinoHardware</plugin>
                 <param name="left_wheel_name">left_wheel_joint</param>
                 <param name="right_wheel_name">right_wheel_joint</param>
                 <param name="loop_rate">30</param>
-                <param name="serial_port">/dev/ttyUSB0</param>
-                <param name="baud_rate">115200</param>
+                <param name="device">/dev/ttyACM0</param>
+                <param name="baud_rate">57600</param>
                 <param name="wheel_radius">0.035</param>
                 <param name="wheel_separation">0.18448</param>
@@ -15,22 +15,22 @@
                 <param name="ppr_right">71.4</param> -->
                 <param name="enc_counts_per_rev">74.3</param>
-                <param name="timeout_ms">1000</param>
+                <param name="timeout_ms">2000</param>
             </hardware>
             <joint name="left_wheel_joint">
+                <state_interface name="position"/>
+                <state_interface name="velocity"/>
                 <command_interface name="velocity">
-                        <param name="min">-10</param>
-                        <param name="max">10</param>
-                    </command_interface>
-                <state_interface name="velocity"/>
-                <state_interface name="position"/>
+                    <param name="min">-10</param>
+                    <param name="max">10</param>
+                </command_interface>
             </joint>
             <joint name="right_wheel_joint">
-                    <command_interface name="velocity">
-                        <param name="min">-10</param>
-                        <param name="max">10</param>
-                    </command_interface>
-                    <state_interface name="velocity"/>
-                    <state_interface name="position"/>
-                </joint>
+                <state_interface name="position"/>
+                <state_interface name="velocity"/>
+                <command_interface name="velocity">
+                    <param name="min">-10</param>
+                    <param name="max">10</param>
+                </command_interface>
+            </joint>
         </ros2_control>
     <!-- </xacro:unless> -->

Commit message: added static transforms

File: src/chassis/description/chassis.urdf.xacro (robot description, xacro)
@@ -9,5 +9,5 @@
         <xacro:include filename="gazebo_control.xacro"/>
     </xacro:if> -->
-    <xacro:include filename="lidar.xacro"/>
+    <!-- <xacro:include filename="lidar.xacro"/> -->
     <!-- <xacro:include filename="camera.xacro"/> -->
 </robot>

File: src/chassis/description/chassis_core.xacro (robot description, xacro)
@@ -118,3 +118,19 @@
         </xacro:inertial_sphere>
     </link>
+    <joint name="lidar_joint" type="fixed">
+        <parent link="base_link"/>
+        <child link="lidar_link"/>
+        <origin xyz="-0.12 0 0.13442" rpy="0 0 0"/>
+    </joint>
+    <link name="lidar_link">
+        <visual>
+            <geometry>
+                <cylinder radius="0.035" length="0.025"/>
+            </geometry>
+            <material name="red"/>
+        </visual>
+        <xacro:inertial_cylinder mass="0.140" length="0.025" radius="0.035">
+            <origin xyz="0 0 0" rpy="0 0 0"/>
+        </xacro:inertial_cylinder>
+    </link>
 </robot>

File: src/chassis/description/lidar.xacro (robot description, xacro)
@@ -1,3 +1,3 @@
-<?xml version="1.0"?>
+<!-- <?xml version="1.0"?>
 <robot xmlns:xacro="http://www.ros.org/wiki/xacro">
     <xacro:include filename="inertial_macros.xacro"/>
@@ -43,3 +43,3 @@
         </sensor>
     </gazebo>
-</robot>
+</robot> -->
