Commit message: updated xacro model

File: src/chassis/description/chassis_core.xacro (robot description, xacro)
@@ -27,18 +27,18 @@
     <link name="chassis_link">
         <visual>
-            <origin xyz="0.13335 0 0.0635" rpy="0 0 0"/>
+            <origin xyz="0.13462 0 0.06096" rpy="0 0 0"/>
             <geometry>
-                <box size="0.2667 0.1651 0.127"/> <!-- 26.67cm x 16.51cm x 12.7cm -->
+                <box size="0.26924 0.1524 0.12192"/>
             </geometry>
             <material name="white"/>
         </visual>
         <collision>
-            <origin xyz="0.13335 0 0.0635" rpy="0 0 0"/>
+            <origin xyz="0.13462 0 0.06096" rpy="0 0 0"/>
             <geometry>
-                <box size="0.2667 0.1651 0.127"/> <!-- 26.67cm x 16.51cm x 12.7cm -->
+                <box size="0.26924 0.1524 0.12192"/>
             </geometry>
         </collision>
-        <xacro:inertial_box mass="0.5" x="0.2667" y="0.1651" z="0.127">
-            <origin xyz="0.13335 0 0.0635" rpy="0 0 0"/>
+        <xacro:inertial_box mass="0.5" x="0.26924" y="0.1524" z="0.12192">
+            <origin xyz="0.13462 0 0.06096" rpy="0 0 0"/>
         </xacro:inertial_box>
     </link>
@@ -47,5 +47,5 @@
         <parent link="base_link"/>
         <child link="left_wheel_link"/>
-        <origin xyz="0 0.096 0" rpy="-1.5707963267948966 0 0"/> <!-- Rotate wheel -->
+        <origin xyz="0 0.09224 -0.0127" rpy="-1.5707963267948966 0 0"/> <!-- Rotate wheel -->
         <axis xyz="0 0 1"/>
     </joint>
@@ -70,5 +70,5 @@
         <parent link="base_link"/>
         <child link="right_wheel_link"/>
-        <origin xyz="0 -0.096 0" rpy="1.5707963267948966 0 0"/> <!-- Rotate wheel -->
+        <origin xyz="0 -0.09224 -0.0127" rpy="1.5707963267948966 0 0"/> <!-- Rotate wheel -->
         <axis xyz="0 0 -1"/>
     </joint>
@@ -98,5 +98,5 @@
         <visual>
             <geometry>
-                <sphere radius="0.035"/>
+                <sphere radius="0.04572"/>
             </geometry>
             <material name="black"/>
@@ -104,9 +104,9 @@
         <collision>
             <geometry>
-                <sphere radius="0.035"/>
+                <sphere radius="0.04572"/>
             </geometry>
             <material name="black"/>
         </collision>
-        <xacro:inertial_sphere mass="0.1" radius="0.035">
+        <xacro:inertial_sphere mass="0.1" radius="0.04572">
             <origin xyz="0 0 0" rpy="0 0 0"/>
         </xacro:inertial_sphere>

File: src/chassis/description/lidar.xacro (robot description, xacro)
@@ -6,5 +6,5 @@
         <parent link="chassis_link"/>
         <child link="lidar_link"/>
-        <origin xyz="0.2 0 0.1395"/>
+        <origin xyz="0.2 0 0.13442"/>
     </joint>
     <link name="lidar_link">

Commit message: fixed mapping

File: src/chassis/description/chassis_core.xacro (robot description, xacro)
@@ -19,4 +19,10 @@
     <!-- BASE LINK -->
     <link name="base_link"></link>
+    <joint name="base_footprint_joint" type="fixed">
+        <parent link="base_link"/>
+        <child link="base_footprint"/>
+        <origin xyz="0 0 0" rpy="0 0 0"/>
+    </joint>
+    <link name="base_footprint"></link>
     <!-- CHASSIS LINK -->
     <joint name="chassis_joint" type="fixed">

File: src/chassis/description/lidar.xacro (robot description, xacro)
@@ -4,7 +4,7 @@
     <!-- LIDAR -->
     <joint name="lidar_joint" type="fixed">
-        <parent link="chassis_link"/>
+        <parent link="base_link"/>
         <child link="lidar_link"/>
-        <origin xyz="0.2 0 0.13442" rpy="0 0 3.14159"/>
+        <origin xyz="0.15 0 0.13442" rpy="0 0 3.14159"/>
     </joint>
     <link name="lidar_link">

File: src/chassis/description/ros2_control.xacro (robot description, xacro)
@@ -7,5 +7,5 @@
                 <param name="left_wheel_name">left_wheel_joint</param>
                 <param name="right_wheel_name">right_wheel_joint</param>
-                <param name="loop_rate">30</param>
+                <param name="loop_rate">10</param>
                 <param name="device">/dev/ttyACM0</param>
                 <param name="baud_rate">57600</param>

Commit message: edited robot dimensions

File: src/chassis/description/chassis_core.xacro (robot description, xacro)
@@ -53,5 +53,5 @@
         <parent link="base_link"/>
         <child link="left_wheel_link"/>
-        <origin xyz="0 0.09224 -0.0127" rpy="-1.5707963267948966 0 0"/> <!-- Rotate wheel -->
+        <origin xyz="0 0.09144 -0.0127" rpy="-1.5707963267948966 0 0"/> <!-- Rotate wheel -->
         <axis xyz="0 0 1"/>
     </joint>
@@ -59,5 +59,5 @@
         <visual>
             <geometry>
-                <cylinder radius="0.035" length="0.027"/>
+                <cylinder radius="0.0325" length="0.027"/>
             </geometry>
             <material name="blue"/>
@@ -65,5 +65,5 @@
         <collision>
             <geometry>
-                <cylinder radius="0.035" length="0.027"/>
+                <cylinder radius="0.0325" length="0.027"/>
             </geometry>
         </collision>
@@ -76,5 +76,5 @@
         <parent link="base_link"/>
         <child link="right_wheel_link"/>
-        <origin xyz="0 -0.09224 -0.0127" rpy="1.5707963267948966 0 0"/> <!-- Rotate wheel -->
+        <origin xyz="0 -0.09144 -0.0127" rpy="1.5707963267948966 0 0"/> <!-- Rotate wheel -->
         <axis xyz="0 0 -1"/>
     </joint>
@@ -82,5 +82,5 @@
         <visual>
             <geometry>
-                <cylinder radius="0.035" length="0.027"/>
+                <cylinder radius="0.0325" length="0.027"/>
             </geometry>
             <material name="blue"/>
@@ -88,5 +88,5 @@
         <collision>
             <geometry>
-                <cylinder radius="0.035" length="0.027"/>
+                <cylinder radius="0.0325" length="0.027"/>
             </geometry>
         </collision>

File: src/chassis/description/ros2_control.xacro (robot description, xacro)
@@ -10,7 +10,7 @@
                 <param name="device">/dev/ttyACM0</param>
                 <param name="baud_rate">57600</param>
-                <param name="wheel_radius">0.035</param>
-                <param name="wheel_separation">0.18448</param>
-                <param name="ppr_left">60.5</param>
+                <param name="wheel_radius">0.0325</param>
+                <param name="wheel_separation">0.18288</param>
+                <param name="ppr_left">70.5</param>
                 <param name="ppr_right">70.5</param>
                 <param name="timeout_ms">2000</param>

Commit message: prep for camera integration

File: src/chassis/description/chassis_core.xacro (robot description, xacro)
@@ -118,8 +118,9 @@
         </xacro:inertial_sphere>
     </link>
+    <!-- LIDAR LINK -->
     <joint name="lidar_joint" type="fixed">
         <parent link="base_link"/>
         <child link="lidar_link"/>
-        <origin xyz="-0.12 0 0.13442" rpy="0 0 0"/>
+        <origin xyz="-0.06 0 0.13442" rpy="0 0 0"/>
     </joint>
     <link name="lidar_link">
@@ -134,3 +135,26 @@
         </xacro:inertial_cylinder>
     </link>
+    <!-- CAMERA LINK -->
+     <joint name="camera_joint" type="fixed">
+        <parent link="base_link"/>
+        <child link="camera_link"/>
+        <origin xyz="-0.11 0.05 0.09" rpy="0 0.785398 0"/>
+    </joint>
+    <link name="camera_link">
+        <visual>
+            <geometry>
+                <box size="0.0076 0.1574 0.0758"/>
+            </geometry>
+            <material name="red"/>
+        </visual>
+        <!-- <xacro:inertial_box mass="0.2" x="0.0076" y="0.1574" z="0.0758">
+            <origin xyz="0 0 0" rpy="0 0 0"/>
+        </xacro:inertial_box> -->
+    </link>
+    <joint name="camera_optical_joint" type="fixed">
+        <parent link="camera_link"/>
+        <child link="camera_optical_link"/>
+        <origin xyz="0 0 0" rpy="-1.5707963267948966 0 -1.5707963267948966"/>
+    </joint>
+    <link name="camera_optical_link"></link>
 </robot>

Commit message: final commit before presentation

File: src/chassis/description/chassis_core.xacro (robot description, xacro)
@@ -142,10 +142,10 @@
     </joint>
     <link name="camera_link">
-        <visual>
+        <!-- <visual>
             <geometry>
                 <box size="0.0076 0.1574 0.0758"/>
             </geometry>
             <material name="red"/>
-        </visual>
+        </visual> -->
         <!-- <xacro:inertial_box mass="0.2" x="0.0076" y="0.1574" z="0.0758">
             <origin xyz="0 0 0" rpy="0 0 0"/>
